File: XC9536_trainer.sch (EAGLE design)
At the start: 7 parts, among them IC1 XC9536_44VQ, U1 FTS31XS-U

Commit message: Changed board size to fit into 5x5cm, added some silkscreen and possibly made it possible to use it in a breadboard.
Parts:
- C1, C2: value (none) -> 0.1µF
Changed lines of the file:
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@@
 <?xml version="1.0" encoding="utf-8"?>
 <!DOCTYPE eagle SYSTEM "eagle.dtd">
-<eagle version="7.1.0">
+<eagle version="7.5.0">
 <drawing>
 <settings>
@@
 <part name="JP1" library="OLED_mod" deviceset="HEADER-1X16" device="ROUND"/>
 <part name="JP2" library="OLED_mod" deviceset="HEADER-1X16" device="ROUND"/>
-<part name="C1" library="rcl" deviceset="C-US" device="C0603K"/>
-<part name="C2" library="rcl" deviceset="C-US" device="C0603K"/>
+<part name="C1" library="rcl" deviceset="C-US" device="C0603K" value="0.1µF"/>
+<part name="C2" library="rcl" deviceset="C-US" device="C0603K" value="0.1µF"/>
 <part name="P+6" library="supply1" deviceset="VCC" device=""/>
 <part name="GND6" library="supply1" deviceset="GND" device=""/>

Commit message: Corrected some silkscreen, adding gerber. Ready for first test production batch.
Parts:
- IC1: value XC9536_44VQ -> XC9536
Changed lines of the file:
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@@
 </classes>
 <parts>
-<part name="IC1" library="xilinx-xc9" deviceset="XC9536_44VQ" device=""/>
+<part name="IC1" library="xilinx-xc9" deviceset="XC9536_44VQ" device="" value="XC9536"/>
 <part name="U1" library="SparkFun-DigitalIC" deviceset="FT231X" device="S" value="FTS31XS-U"/>
 <part name="CN1" library="OLED_mod" deviceset="USB" device="MINIBLARGE"/>
